Commit message: Spawning elements correctly

File: sr_taco_launch/other/base_with_kinect.urdf.xacro (robot description, xacro)
@@ -2,5 +2,5 @@
   <include filename="$(find sr_description)/materials.urdf.xacro" />
   <include filename="$(find sr_taco_launch)/other/xacro/kinect/kinect.urdf.xacro" />
-  <include filename="$(find sr_taco_launch)/other/xacro/desk/desk.urdf.xacro" />
+  <include filename="$(find sr_taco_launch)/other/xacro/desk/desk2.urdf.xacro" />
   <xacro:desk/>
   <xacro:base_mounted_kinect parent="desk2_pillar">

File: sr_taco_launch/other/xacro/desk/desk2.urdf.xacro (robot description, xacro)
@@ -1,25 +1,25 @@
 <robot name="desk" xmlns:body="http://playerstage.sourceforge.net/gazebo/xmlschema/#body" xmlns:geom="http://playerstage.sourceforge.net/gazebo/xmlschema/#geom" xmlns:interface="http://playerstage.sourceforge.net/gazebo/xmlschema/#interface" xmlns:joint="http://playerstage.sourceforge.net/gazebo/xmlschema/#slider" xmlns:xacro="http://ros.org/wiki/xacro">
   <xacro:macro name="desk">
-  <link name="desk_pillar">
+  <link name="desk2_pillar">
     <inertial>
-      <origin xyz="0 0 0.5"/>
+      <origin xyz="0 0 0.75"/>
       <mass value="1000.0"/>
       <inertia ixx="1.0" ixy="0.0" ixz="0.0" iyy="1.0" iyz="0.0" izz="1.0"/>
     </inertial>
     <visual>
-      <origin rpy="0 0 0" xyz="0 0 0.51"/>
+      <origin rpy="0 0 0" xyz="0 0 0.76"/>
       <geometry name="desk_visual">
-        <cylinder length="0.98" radius="0.1"/>
+        <cylinder length="1.48" radius="0.1"/>
       </geometry>
       <material name="Green"/>
     </visual>
     <collision>
-      <origin rpy="0 0 0" xyz="0 0 0.51"/>
+      <origin rpy="0 0 0" xyz="0 0 0.76"/>
       <geometry name="desk_collision">
-        <cylinder length=".98" radius="0.1"/>
+        <cylinder length="1.48" radius="0.1"/>
       </geometry>
     </collision>
   </link>
-  <gazebo reference="desk_pillar">
+  <gazebo reference="desk2_pillar">
     <material>Gazebo/Green</material>
     <mu1>1000.0</mu1>
@@ -29,5 +29,5 @@
     <selfCollide>true</selfCollide>
   </gazebo>
-  <link name="desk_support">
+  <link name="desk2_support">
     <inertial>
       <origin xyz="0 0 0"/>
@@ -38,5 +38,5 @@
       <origin rpy="0 0 0" xyz="0 0 0.01"/>
       <geometry name="desk_s_visual">
-        <cylinder length="0.02" radius="0.2"/>
+        <cylinder length="0.02" radius="1.0"/>
       </geometry>
       <material name="Green"/>
@@ -45,9 +45,9 @@
       <origin rpy="0 0 0" xyz="0 0 0.01"/>
       <geometry name="desk_s_collision">
-        <cylinder length="0.02" radius="0.2"/>
+        <cylinder length="0.02" radius="1.0"/>
       </geometry>
     </collision>
   </link>
-  <gazebo reference="desk_support">
+  <gazebo reference="desk2_support">
     <material>Gazebo/Green</material>
     <mu1>1000.0</mu1>
@@ -56,9 +56,8 @@
     <kd>1.0</kd>
     <selfCollide>true</selfCollide>
-    <static>true</static>
   </gazebo>
   <joint name="desk_joint" type="fixed">
-    <parent link="desk_support"/>
-    <child link="desk_pillar"/>
+    <parent link="desk2_support"/>
+    <child link="desk2_pillar"/>
     <origin rpy="0 0 0" xyz="0 0 0.02"/>
   </joint>

File: sr_taco_launch/other/xacro/objects/table.urdf.xacro (robot description, xacro)
@@ -17,5 +17,5 @@
   <property name="table_depth" value="0.70" />
   <property name="leg_radius" value="0.02" />
-  <property name="table_x" value="0.0" />
+  <property name="table_x" value="0.98" />
   <property name="table_y" value="0.0" />
   <property name="table_z" value="0.0" />
@@ -25,5 +25,5 @@
   <link name="table_top_link">
     <inertial>
-      <mass value="1.0" />
+      <mass value="20.0" />
       <origin xyz="${table_x} ${table_y} ${table_z+table_height-table_top_thickness/2}" />
       <inertia ixx="1" ixy="0"  ixz="0"
@@ -58,5 +58,5 @@
   <link name="leg1_link">
     <inertial>
-      <mass value="1.0" />
+      <mass value="10.0" />
       <origin xyz="0 0 ${-table_height/2}" />
       <inertia ixx="0.1" ixy="0"  ixz="0"
@@ -92,5 +92,5 @@
   <link name="leg2_link">
     <inertial>
-      <mass value="1.0" />
+      <mass value="10.0" />
       <origin xyz="0 0 ${-table_height/2}" />
       <inertia ixx="0.1" ixy="0"  ixz="0"
@@ -126,5 +126,5 @@
   <link name="leg3_link">
     <inertial>
-      <mass value="1.0" />
+      <mass value="10.0" />
       <origin xyz="0 0 ${-table_height/2}" />
       <inertia ixx="0.1" ixy="0"  ixz="0"
@@ -160,5 +160,5 @@
   <link name="leg4_link">
     <inertial>
-      <mass value="1.0" />
+      <mass value="10.0" />
       <origin xyz="0 0 ${-table_height/2}" />
       <inertia ixx="0.1" ixy="0"  ixz="0"
@@ -188,5 +188,6 @@
   </gazebo>
   <gazebo>
-    <static>true</static>
+    <!--static>true</static-->
+    <turnGravityOff>false</turnGravityOff>
     <canonicalBody>table_top_link</canonicalBody>
   </gazebo>

File: sr_taco_launch/robots/arm_and_hand_motor.urdf.xacro (robot description, xacro)
@@ -4,5 +4,5 @@
   <include filename="$(find sr_description)/hand/xacro/full_hand_motor.urdf.xacro" />
   <include filename="$(find sr_description)/other/xacro/gazebo/gazebo.urdf.xacro" />
-  <include filename="$(find sr_description)/other/xacro/desk/desk.urdf.xacro" />
+  <include filename="$(find sr_taco_launch)/other/xacro/desk/desk.urdf.xacro" />
   <xacro:desk/>
   <joint name="arm_to_desk_fixed" type="fixed">
