Commit message: Desk no longer included in the robot_model for the arm and hand, because otherwise some planning nodes crash.

File: sr_taco_launch/other/xacro/desk/desk.urdf.xacro (robot description, xacro)
@@ -56,5 +56,5 @@
     <kd>1.0</kd>
     <selfCollide>true</selfCollide>
-    <static>true</static>
+    <!--static>true</static-->
   </gazebo>
   <joint name="desk_joint" type="fixed">

File: sr_taco_launch/robots/arm_and_hand_motor.urdf.xacro (robot description, xacro)
@@ -4,8 +4,7 @@
   <include filename="$(find sr_description)/hand/xacro/full_hand_motor.urdf.xacro" />
   <include filename="$(find sr_description)/other/xacro/gazebo/gazebo.urdf.xacro" />
-  <include filename="$(find sr_taco_launch)/other/xacro/desk/desk.urdf.xacro" />
-  <xacro:desk/>
-  <joint name="arm_to_desk_fixed" type="fixed">
-    <parent link="desk_pillar"/>
+  <link name="world" />
+  <joint name="arm_to_world_fixed" type="fixed">
+    <parent link="world"/>
     <child link="shadowarm_base"/>
     <origin rpy="0 0 0" xyz="0 0 1.0"/>
