Commit message: throwing the lid opened at the end

File: sr_taco_launch/other/xacro/objects/suitcase.urdf.xacro (robot description, xacro)
@@ -190,5 +190,5 @@
   <joint name="lid_joint" type="revolute" >
     <axis xyz="0 -1 0"/>
-    <limit effort="1000.0" lower="${M_PI/2}" upper="${M_PI}" velocity="0.5"/>
+    <limit effort="1000.0" lower="0.2" upper="${M_PI}" velocity="0.5"/>
     <parent link="wall1_link" />
     <!--origin xyz="${suitcase_x+suitcase_width/2} ${suitcase_y} ${suitcase_z+suitcase_height}" rpy="0 0 0" /-->
